Commit message: Second push

File: ur_description/urdf/ur10_new.urdf (robot description, URDF)
Before this commit: robot ur10, 11 links, 10 joints
Links:
- link base_link: geometry collision mesh filename=package://ur_description/meshes/ur10/collision/base.stl; visual mesh filename=package://ur_description/meshes/ur10/visual/base.stl
- link forearm_link: geometry collision mesh filename=package://ur_description/meshes/ur10/collision/forearm.stl; visual mesh filename=package://ur_description/meshes/ur10/visual/forearm.stl
- link shoulder_link: geometry collision mesh filename=package://ur_description/meshes/ur10/collision/shoulder.stl; visual mesh filename=package://ur_description/meshes/ur10/visual/shoulder.stl
- link upper_arm_link: geometry collision mesh filename=package://ur_description/meshes/ur10/collision/upperarm.stl; visual mesh filename=package://ur_description/meshes/ur10/visual/upperarm.stl
- link wrist_1_link: geometry collision mesh filename=package://ur_description/meshes/ur10/collision/wrist1.stl; visual mesh filename=package://ur_description/meshes/ur10/visual/wrist1.stl
- link wrist_2_link: geometry collision mesh filename=package://ur_description/meshes/ur10/collision/wrist2.stl; visual mesh filename=package://ur_description/meshes/ur10/visual/wrist2.stl
- link wrist_3_link: geometry collision mesh filename=package://ur_description/meshes/ur10/collision/wrist3.stl; visual mesh filename=package://ur_description/meshes/ur10/visual/wrist3.stl
